File: veittur-p1-ble.kicad_pcb (KiCad board)
At the start: 2 copper layers, 40 x 20 mm, 21 parts, among them J1 Connector_HAN_P1, J2 Conn_01x06, Q1 BSS138, Q2 BSS138, U1 MIC5504-3.3YM5, U2 CH582F, U3 74AHCT1G125, Y1 32M, Y2 32k

Commit message: initial "complete"
is that it? should I just order this then?
Parts:
- removed R3: 10k, Resistor_SMD:R_0603_1608Metric
- removed U3: 74AHCT1G125, Package_TO_SOT_SMD:SOT-23-5
- AE1: value Antenna_Dipole -> Antenna_Loop; footprint RF_Antenna:Texas_SWRA117D_2.4GHz_Right -> wch-antenna:ANT-F-1-2.4G-1.6MM-FR4-WCH-FLIP
- D1: value WS2812B -> WS2812C-2020; footprint LED_SMD:LED_WS2812B_PLCC4_5.0x5.0mm_P3.2mm -> LED_SMD:LED_WS2812-2020-PLCC4_2.0x2.0mm
- moved D1 6.24 mm to (120.6, 82.1), turned to -90 degrees
- moved AE1 5.05 mm to (136.9, 88.1)
- moved C3 0.54 mm to (126.5, 86.0)
Connections:
- D1 pad 1: +5V -> unconnected-(D1-Pad1)
- D1 pad 2: unconnected-(D1-Pad2) -> GND
- D1 pad 3: GND -> /LED_OUT3V3
- D1 pad 4: /LED_OUT5V -> +5V
- U2 pad 29: (no net) -> GND
Routing:
- net +5V: track 54.8 -> 45.8 mm
- net /LED_OUT5V: track 2.52 -> 0.00 mm
- net /LED_ENABLE: track 1.91 -> 0.00 mm
- net GND: vias 0 -> 38
Other:
- board text added: "+5"
- board text added: "3V3"
- board text added: "G"
- board text added: "GND"
- board text added: "JLCJLCJLCJLC"
- board text added: "OUT"
- board text added: "RQ"
- board text added: "RX"
- board text added: "Serial Meter#"
- board text added: "TCK"
- board text added: "TIO"
- board text added: "TX"
- board text removed: "3V3 GND RX TX TIO TCK"
